File: sag-split.sch (KiCad schematic (older format))
At the start: 16 parts

Commit message: added footprints
Parts:
- added D1, D2, D3, D4: SOD-123, Diode_SMD:D_SOD-123, symbol Device:D_Small
- added MX1, MX2, MX3: MX-NoLED, MX_Alps_Hybrid:MX-1U, symbol MX_Alps_Hybrid:MX-NoLED
- added MX4: MX-NoLED, Resistor_SMD:R_0805_2012Metric, symbol MX_Alps_Hybrid:MX-NoLED
- C1, C2, C3, C4, C5, C6, C7: renamed from C?; footprint (none) -> Capacitor_SMD:C_0805_2012Metric
- F1: renamed from F?; footprint (none) -> Fuse:Fuse_1206_3216Metric
- R1, R2, R3, R4: renamed from R?; footprint (none) -> Resistor_SMD:R_0805_2012Metric
- SW1: renamed from SW?; footprint (none) -> random-keyboard-parts:SKQG-1155865
- USB1: renamed from USB?; footprint (none) -> random-keyboard-parts:Molex-0548190589
- Y1: renamed from Y?; footprint (none) -> Crystal:Crystal_SMD_3225-4Pin_3.2x2.5mm
- gave numbers to parts that had none: 1
Connections:
- new net: D1.2 (A), MX1.2 (ROW)
- new net: D3.2 (A), MX3.2 (ROW)
- new net: D4.2 (A), MX4.2 (ROW)
- new net: D2.2 (A), MX2.2 (ROW)
- new net COL0: MX1.1 (COL), MX2.1 (COL)
- new net COL1: MX3.1 (COL), MX4.1 (COL)
- new net ROW0: D1.1 (K), D3.1 (K)
- new net ROW1: D2.1 (K), D4.1 (K)
